File: Lesson 4/Eagle/DIYpiano/DIYpiano.sch (EAGLE design)
At the start: 21 parts, among them IC1 NE555N, SW1 MOMENTARY-SWITCH-SPST-PTH-6.0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, SW2 MOMENTARY-SWITCH-SPST-PTH-6.0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, SW3 MOMENTARY-SWITCH-SPST-PTH-6.0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, SW4 MOMENTARY-SWITCH-SPST-PTH-6.0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, SW5 MOMENTARY-SWITCH-SPST-PTH-6.0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, SW6 MOMENTARY-SWITCH-SPST-PTH-6.0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, SW7 MOMENTARY-SWITCH-SPST-PTH-6.0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, SW8 MOMENTARY-SWITCH-SPST-PTH-6.0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

Commit message: Completed SCH
.
Parts:
- removed JP1: (no value), pinhead:PINHD-1X2
- added BATT: 3V, adafruit:CR1220THM
- added C2: 100nF, rcl:C-US025-025X050
- added Q1: 2N2222, transistor:-NPN-TO92-E1
- added R10: 910, rcl:R-US_0207/10
- C1: value 100n -> 100nF
- IC1: MPN (none) -> TLC555CP; OC_NEWARK unknown -> 24M8296
- LS1: value BUZZER-PTH_NO_SILK -> AT-1220-TT-3V-2-R; device SparkFun-Electromechanical:BUZZER-PTH_NO_SILK -> buzzer:F/HMB; OC_NEWARK unknown -> (none)
- R3: value 390 -> 1K
- R4: value 910 -> 390
- R5: value 1K -> 1.5K
- R6: value 1.1K -> 1.3K
- R8: value 1.3K -> 1.1K
- R9: value 1.5K -> 1K
Connections:
- new net N$12: C2.1, IC1.CV
- new net N$13: LS1.-, Q1.C
- new net N$14: Q1.B, R1.1
- net GND: now also BATT.-, C2.2, Q1.E; no longer JP1.1, LS1.2
- net N$1: now also R4.1, SW2.2; no longer R3.1, SW1.2
- net N$10: now also R5.2, SW1.2; no longer R9.2, SW8.2
- net N$11: now also R1.2; no longer LS1.1
- net N$2: now also R3.1; no longer R1.1
- net N$4: now also R10.1, R4.2, SW8.2; no longer R3.2, R4.1, SW2.2
- net N$5: now also R10.2, R9.1, SW7.2; no longer R4.2, R5.1, SW3.2
- net N$6: now also R8.1, R9.2, SW6.2; no longer R5.2, R6.1, SW4.2
- net N$7: now also R8.2; no longer R6.2
- net N$8: now also R6.1, SW4.2; no longer R8.1, SW6.2
- net N$9: now also R5.1, R6.2, SW3.2; no longer R8.2, R9.1, SW7.2
- net VCC: now also BATT.+, BATT.+1, LS1.+, R3.2; no longer JP1.2, R1.2
Other:
- moved on the sheet: R1, R3, R4, R5, R6, R8, R9, SW1, SW2, SW3, SW4, SW6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
